File: 0101-PUSH.kicad_pcb (KiCad board)
At the start: 2 copper layers, 24.6 x 19.6 mm, 14 parts, among them J1 Conn_01x03, SW1 PUSH

Commit message: Rework with new design
Parts:
- removed H1, H2: MountingHole, MountingHole:MountingHole_2.2mm_M2
- removed kibuzzard-631DB129: G***, kibuzzard-631DB129
- removed kibuzzard-631DDE16: G***, kibuzzard-631DDE16
- added kibuzzard-6324301C: G***, kibuzzard-6324301C, F.Cu at (110.0, 106.5)
- added kibuzzard-63243463: G***, kibuzzard-63243463, F.Cu at (115.5, 112.5)
- added kibuzzard-63243468: G***, kibuzzard-63243468, F.Cu at (117.0, 112.5)
- added kibuzzard-63243772: G***, kibuzzard-63243772, F.Cu at (116.2, 108.5)
- added kibuzzard-63243779: G***, kibuzzard-63243779, F.Cu at (116.2, 116.5)
- added kibuzzard-632ECE43: G***, kibuzzard-632ECE43, F.Cu at (102.5, 118.5)
- R1, R2, R3, R4: footprint Resistor_SMD:R_0402_1005Metric -> Resistor_SMD:R_0603_1608Metric
- moved C1 14.5 mm to (118.5, 114.9), turned to 90 degrees
- moved R2 13.1 mm to (117.0, 114.6), turned to 90 degrees
- moved R4 13.0 mm to (117.0, 110.4), turned to -90 degrees
- moved D1 12.3 mm to (104.0, 115.0)
- moved R1 11.7 mm to (115.5, 114.6), turned to -90 degrees
- moved R3 11.5 mm to (115.5, 110.4), turned to 90 degrees
- moved R5 11.3 mm to (104.5, 112.5), turned to 0 degrees
- moved J1 5.10 mm to (107.5, 104.0), turned to 90 degrees
Connections:
- SW1 pad 2: VCC -> /KEY
- SW1 pad 3: Net-(R5-Pad2) -> Net-(R3-Pad2)
- SW1 pad 5: /KEY -> Net-(R5-Pad2)
- SW1 pad 6: Net-(R3-Pad2) -> VCC
Routing:
- net VCC: track 24.0 -> 17.5 mm, vias 1 -> 0
- net /KEY: track 14.4 -> 17.3 mm
- net Net-(R3-Pad2): track 3.80 -> 4.47 mm
- net GND: vias 28 -> 26
Other:
- board size 24.6 x 19.6 mm -> 19.6 x 19.6 mm
