File: 0101-PUSH.kicad_sch (KiCad schematic)
At the start: 11 parts

Commit message: Finish
Parts:
- C1: value (none) -> 0.1uF(NC); footprint (none) -> Capacitor_SMD:C_0402_1005Metric
- D1: value (none) -> LED; footprint (none) -> LED_SMD:LED_0603_1608Metric; Manufacturer (none) -> EVERLIGHT; PartNumber (none) -> C72041; Supplier (none) -> JLC
- H1, H2: value (none) -> MountingHole; footprint (none) -> MountingHole:MountingHole_2.2mm_M2
- J1: value (none) -> Conn_01x03; footprint (none) -> Connector_PinHeader_2.54mm:PinHeader_1x03_P2.54mm_Vertical
- R1, R2: value (none) -> 10K(NC); footprint (none) -> Resistor_SMD:R_0402_1005Metric
- R3, R4: value (none) -> 0R(NC); footprint (none) -> Resistor_SMD:R_0402_1005Metric
- R5: value (none) -> 2K; footprint (none) -> Resistor_SMD:R_0402_1005Metric; Manufacturer (none) -> UniOhm; PartNumber (none) -> C4109; Supplier (none) -> JLC
- SW1: value (none) -> PUSH; footprint (none) -> JLC-SMT:SW_Push_DPDT_8.5x8.5mm; Manufacturer (none) -> GANGYUAN; PartNumber (none) -> C194405; Supplier (none) -> JLC-EXT

Commit message: Update pull-up/down resistors
Parts:
- R1: value 10K(NC) -> 10K; Manufacturer (none) -> UniOhm; PartNumber (none) -> C25744; Supplier (none) -> JLC
- R4: value 0R(NC) -> 0R; Manufacturer (none) -> UniOhm; PartNumber (none) -> C17168; Supplier (none) -> JLC
Changed lines of the file:
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@@
       (effects (font (size 1.27 1.27)) (justify left))
     )
-    (property "Value" "10K(NC)" (id 1) (at 83.0072 93.853 0)
+    (property "Value" "10K" (id 1) (at 83.0072 93.853 0)
       (effects (font (size 1.27 1.27)) (justify left))
     )
@@
       (effects (font (size 1.27 1.27)) hide)
     )
-    (property "Manufacturer" "~" (id 4) (at 81.28 92.71 0)
-      (effects (font (size 1.27 1.27)) hide)
-    )
-    (property "PartNumber" "~" (id 5) (at 81.28 92.71 0)
-      (effects (font (size 1.27 1.27)) hide)
-    )
-    (property "Supplier" "~" (id 6) (at 81.28 92.71 0)
+    (property "Manufacturer" "UniOhm" (id 4) (at 81.28 92.71 0)
+      (effects (font (size 1.27 1.27)) hide)
+    )
+    (property "PartNumber" "C25744" (id 5) (at 81.28 92.71 0)
+      (effects (font (size 1.27 1.27)) hide)
+    )
+    (property "Supplier" "JLC" (id 6) (at 81.28 92.71 0)
       (effects (font (size 1.27 1.27)) hide)
     )
@@
       (effects (font (size 1.27 1.27)) (justify left))
     )
-    (property "Value" "0R(NC)" (id 1) (at 103.3272 106.553 0)
+    (property "Value" "0R" (id 1) (at 103.3272 106.553 0)
       (effects (font (size 1.27 1.27)) (justify left))
     )
@@
       (effects (font (size 1.27 1.27)) hide)
     )
-    (property "Manufacturer" "~" (id 4) (at 101.6 105.41 0)
-      (effects (font (size 1.27 1.27)) hide)
-    )
-    (property "PartNumber" "~" (id 5) (at 101.6 105.41 0)
-      (effects (font (size 1.27 1.27)) hide)
-    )
-    (property "Supplier" "~" (id 6) (at 101.6 105.41 0)
+    (property "Manufacturer" "UniOhm" (id 4) (at 101.6 105.41 0)
+      (effects (font (size 1.27 1.27)) hide)
+    )
+    (property "PartNumber" "C17168" (id 5) (at 101.6 105.41 0)
+      (effects (font (size 1.27 1.27)) hide)
+    )
+    (property "Supplier" "JLC" (id 6) (at 101.6 105.41 0)
       (effects (font (size 1.27 1.27)) hide)
     )
@@
     )
     (path "/00000000-0000-0000-0000-0000631b4f4a"
-      (reference "R1") (unit 1) (value "10K(NC)") (footprint "Resistor_SMD:R_0402_1005Metric")
+      (reference "R1") (unit 1) (value "10K") (footprint "Resistor_SMD:R_0402_1005Metric")
     )
     (path "/00000000-0000-0000-0000-0000631b60c2"
@@
     )
     (path "/00000000-0000-0000-0000-0000631c3840"
-      (reference "R4") (unit 1) (value "0R(NC)") (footprint "Resistor_SMD:R_0402_1005Metric")
+      (reference "R4") (unit 1) (value "0R") (footprint "Resistor_SMD:R_0402_1005Metric")
     )
     (path "/00000000-0000-0000-0000-0000631bf244"

Commit message: Rework with new design
Parts:
- removed H1, H2: MountingHole, MountingHole:MountingHole_2.2mm_M2, symbol Mechanical:MountingHole
- R1: footprint Resistor_SMD:R_0402_1005Metric -> Resistor_SMD:R_0603_1608Metric; Manufacturer UniOhm -> UNI-ROYAL; PartNumber C25744 -> C25804
- R2, R3: footprint Resistor_SMD:R_0402_1005Metric -> Resistor_SMD:R_0603_1608Metric
- R4: footprint Resistor_SMD:R_0402_1005Metric -> Resistor_SMD:R_0603_1608Metric; Manufacturer UniOhm -> UNI-ROYAL; PartNumber C17168 -> C21189
- R5: Manufacturer UniOhm -> UNI-ROYAL
Connections:
- net KEY: now also SW1.2 (B); no longer SW1.5 (B)
- net VCC: now also SW1.6 (C); no longer SW1.2 (B)
- net at SW1.3 (C): now also R3.2, R4.1; no longer R5.2
- new net: R5.2, SW1.5 (B)
Other:
- moved on the sheet: C1, D1, R1, R2, R3, R4, R5
